Commit message: remove green

File: mcr_common/mcr_description/urdf/materials.urdf.xacro (robot description, xacro)
@@ -3,7 +3,4 @@
   <material name="Blue">
     <color rgba="0.0 0.0 0.8 1.0"/>
-  </material>
-  <material name="Green">
-    <color rgba="0.0 0.8 0.0 1.0"/>
   </material>
   <material name="Grey">

Commit message: remove colors

File: mcr_common/mcr_description/urdf/materials.urdf.xacro (robot description, xacro)
@@ -3,7 +3,4 @@
   <material name="Blue">
     <color rgba="0.0 0.0 0.8 1.0"/>
-  </material>
-  <material name="Grey">
-    <color rgba="0.7 0.7 0.7 1.0"/>
   </material>
   <material name="Grey2">
@@ -12,13 +9,4 @@
   <material name="LightGrey">
     <color rgba="0.82 0.82 0.82 1.0"/>
-  </material>
-  <material name="Red">
-    <color rgba="0.8 0.0 0.0 1.0"/>
-  </material>
-  <material name="White">
-    <color rgba="1.0 1.0 1.0 1.0"/>
-  </material>
-  <material name="Black">
-    <color rgba="0.0 0.0 0.0 1.0"/>
   </material>
   <material name="Caster">

Commit message: modified xacro includes

File: mcr_common/mcr_description/urdf/materials.urdf.xacro (robot description, xacro)
@@ -26,14 +26,14 @@
   </material>
   <material name="Caster">
-    <texture filename="package://pr2_ogre/Media/materials/textures/pr2_caster_texture.png" />
+    <texture filename="package://pr2_description/materials/textures/pr2_caster_texture.png" />
   </material>
   <material name="Wheel_l">
-    <texture filename="package://pr2_ogre/Media/materials/textures/pr2_wheel_left.png" />
+    <texture filename="package://pr2_description/materials/textures/pr2_wheel_left.png" />
   </material>
   <material name="Wheel_r">
-    <texture filename="package://pr2_ogre/Media/materials/textures/pr2_wheel_right.png" />
+    <texture filename="package://pr2_description/materials/textures/pr2_wheel_right.png" />
   </material>
   <material name="RollLinks">
-    <texture filename="package://pr2_ogre/Media/materials/textures/pr2_wheel_left.png" />
+    <texture filename="package://pr2_description/materials/textures/pr2_wheel_left.png" />
   </material>
 </root>

File: mcr_common/mcr_description/urdf/ptu/ptu46.transmission.xacro (robot description, xacro)
@@ -2,13 +2,19 @@
 <robot xmlns:xacro="http://ros.org/wiki/xacro">
 	<xacro:macro name="ptu46_transmission" params="name">
-		<transmission name="${name}_pan_trans" type="pr2_mechanism_model/SimpleTransmission">
-			<actuator name="${name}_pan_motor"/>
-			<joint name="${name}_pan_joint"/>
-			<mechanicalReduction>1</mechanicalReduction>
+		<transmission name="${name}_pan_trans">
+		        <type>transmission_interface/SimpleTransmission</type>
+			<actuator name="${name}_pan_motor">
+			  <mechanicalReduction>1</mechanicalReduction>
+			  <hardwareInterface>EffortJointInterface</hardwareInterface>
+			</actuator>
+                        <joint name="${name}_pan_joint"/>
 		</transmission>
-		<transmission name="${name}_tilt_trans" type="pr2_mechanism_model/SimpleTransmission">
-			<actuator name="${name}_tilt_motor"/>
+		<transmission name="${name}_tilt_trans">
+		        <type>transmission_interface/SimpleTransmission</type>
+			<actuator name="${name}_tilt_motor">
+			  <mechanicalReduction>1</mechanicalReduction>
+			  <hardwareInterface>EffortJointInterface</hardwareInterface>
+			</actuator>
 			<joint name="${name}_tilt_joint"/>
-			<mechanicalReduction>1</mechanicalReduction>
 		</transmission>
 	</xacro:macro>

File: mcr_common/mcr_description/urdf/ptu/ptu46.urdf.xacro (robot description, xacro)
@@ -1,6 +1,6 @@
 <?xml version="1.0"?>
 <robot xmlns:xacro="http://ros.org/wiki/xacro">
-	<include filename="$(find mcr_description)/urdf/ptu/ptu46.gazebo.xacro" />
-	<include filename="$(find mcr_description)/urdf/ptu/ptu46.transmission.xacro" />
+	<xacro:include filename="$(find mcr_description)/urdf/ptu/ptu46.gazebo.xacro" />
+	<xacro:include filename="$(find mcr_description)/urdf/ptu/ptu46.transmission.xacro" />
 	<xacro:macro name="ptu46" params="parent name *origin">
 		<link name="${name}_link">

File: mcr_common/mcr_description/urdf/sensors/asus_xtion_camera.urdf.xacro (robot description, xacro)
@@ -1,5 +1,5 @@
 <?xml version="1.0"?>
 <root xmlns:xacro="http://playerstage.sourceforge.net/gazebo/xmlschema/#interface">
-  <include filename="$(find mcr_description)/urdf/sensors/asus_xtion_camera.gazebo.xacro" />
+  <xacro:include filename="$(find mcr_description)/urdf/sensors/asus_xtion_camera.gazebo.xacro" />
   <property name="eye_x_offset" value="0.03" />
   <property name="eye_y_offset" value="0.035" />

File: mcr_common/mcr_description/urdf/sensors/hokuyo_lx30.urdf.xacro (robot description, xacro)
@@ -4,5 +4,5 @@
        xmlns:interface="http://playerstage.sourceforge.net/gazebo/xmlschema/#interface"
        xmlns:xacro="http://ros.org/wiki/xacro">
-  <include filename="$(find mcr_description)/urdf/sensors/hokuyo_lx30.gazebo.xacro" />
+  <xacro:include filename="$(find mcr_description)/urdf/sensors/hokuyo_lx30.gazebo.xacro" />
   <xacro:macro name="hokuyo_lx30" params="name parent *origin ros_topic update_rate min_angle max_angle">
     <joint name="${name}_joint" type="fixed">

File: mcr_common/mcr_description/urdf/sensors/kinect_camera.urdf.xacro (robot description, xacro)
@@ -4,5 +4,5 @@
       xmlns:interface="http://playerstage.sourceforge.net/gazebo/xmlschema/#interface"
       xmlns:xacro="http://ros.org/wiki/xacro">
-  <include filename="$(find mcr_description)/urdf/sensors/kinect_camera.gazebo.xacro" />
+  <xacro:include filename="$(find mcr_description)/urdf/sensors/kinect_camera.gazebo.xacro" />
   <xacro:macro name="kinect_camera" params="name parent *origin">
     <joint name="${name}_frame_joint" type="fixed">

File: mcr_common/mcr_description/urdf/sensors/microsoft_lifecam.urdf.xacro (robot description, xacro)
@@ -4,5 +4,5 @@
       xmlns:interface="http://playerstage.sourceforge.net/gazebo/xmlschema/#interface"
       xmlns:xacro="http://ros.org/wiki/xacro">
-  <include filename="$(find mcr_description)/urdf/sensors/microsoft_lifecam.gazebo.xacro"/>
+  <xacro:include filename="$(find mcr_description)/urdf/sensors/microsoft_lifecam.gazebo.xacro"/>
   <xacro:macro name="microsoft_lifecam" params="name parent *origin">
    <joint name="${name}_camera_joint" type="fixed">

File: mcr_common/mcr_description/urdf/sensors/pmd_camboard_nano_camera.urdf.xacro (robot description, xacro)
@@ -4,5 +4,5 @@
       xmlns:interface="http://playerstage.sourceforge.net/gazebo/xmlschema/#interface"
       xmlns:xacro="http://ros.org/wiki/xacro">
-  <include filename="$(find mcr_description)/urdf/sensors/pmd_camboard_nano_camera.gazebo.xacro" />
+  <xacro:include filename="$(find mcr_description)/urdf/sensors/pmd_camboard_nano_camera.gazebo.xacro" />
   <xacro:macro name="pmd_camboard_nano_camera" params="name parent *origin">
     <joint name="${name}_frame_joint" type="fixed">

File: mcr_common/mcr_description/urdf/sensors/sick_lms_200.urdf.xacro (robot description, xacro)
@@ -1,5 +1,5 @@
 <?xml version="1.0"?>
 <robot xmlns:xacro="http://ros.org/wiki/xacro">
-	<include filename="$(find mcr_description)/urdf/sensors/sick_lms_200.gazebo.xacro" />
+	<xacro:include filename="$(find mcr_description)/urdf/sensors/sick_lms_200.gazebo.xacro" />
 	<xacro:macro name="sick_lms_200" params="name parent *origin ros_topic update_rate min_angle max_angle">
 		<joint name="${name}_joint" type="fixed">

File: mcr_environments/mcr_gazebo_objects/ros/templates/screw.urdf.xacro (robot description, xacro)
@@ -1,6 +1,6 @@
 <?xml version="1.0"?>
 <robot name="screw_template" xmlns:xacro="http://ros.org/wiki/xacro">
-	<include filename="$(find mcr_gazebo_objects)/ros/templates/pipe.urdf.xacro" />
-	<include filename="$(find mcr_gazebo_objects)/ros/templates/nut.urdf.xacro" />
+	<xacro:include filename="$(find mcr_gazebo_objects)/ros/templates/pipe.urdf.xacro" />
+	<xacro:include filename="$(find mcr_gazebo_objects)/ros/templates/nut.urdf.xacro" />
 	<xacro:macro name="screw_template" params="name length radius color">
 		<xacro:pipe_template name="pipe_20" radius="${radius / 2}" height="${length}" color="Gazebo/Black" />

File: mcr_environments/mcr_gazebo_objects/ros/urdf/adapter_sleeve_r20.urdf.xacro (robot description, xacro)
@@ -1,5 +1,5 @@
 <?xml version="1.0"?>
 <robot name="adapter_sleeve_r20" xmlns:xacro="http://ros.org/wiki/xacro">
-	<include filename="$(find mcr_gazebo_objects)/ros/templates/model.urdf.xacro" />
+	<xacro:include filename="$(find mcr_gazebo_objects)/ros/templates/model.urdf.xacro" />
 	<xacro:model_template name="adapter_sleeve_r20" model_filename="adapter_sleeve_r20.dae" scale="0.001" size_x="0.03" size_y="0.03" size_z="0.045" weight="0.010"/>
 </robot>

File: mcr_environments/mcr_gazebo_objects/ros/urdf/adapter_sleeve_v20.urdf.xacro (robot description, xacro)
@@ -1,5 +1,5 @@
 <?xml version="1.0"?>
 <robot name="adapter_sleeve_v20" xmlns:xacro="http://ros.org/wiki/xacro">
-	<include filename="$(find mcr_gazebo_objects)/ros/templates/model.urdf.xacro" />
+	<xacro:include filename="$(find mcr_gazebo_objects)/ros/templates/model.urdf.xacro" />
 	<xacro:model_template name="adapter_sleeve_v20" model_filename="adapter_sleeve_v20.dae" scale="0.001" size_x="0.03" size_y="0.03" size_z="0.045" weight="0.015"/>
 </robot>

File: mcr_environments/mcr_gazebo_objects/ros/urdf/aluprofil_f20_100_gray.urdf.xacro (robot description, xacro)
@@ -1,5 +1,5 @@
 <?xml version="1.0"?>
 <robot name="aluprofil_f20_100_gray" xmlns:xacro="http://ros.org/wiki/xacro">
-	<include filename="$(find mcr_gazebo_objects)/ros/templates/model.urdf.xacro" />
+	<xacro:include filename="$(find mcr_gazebo_objects)/ros/templates/model.urdf.xacro" />
 	<xacro:model_template name="aluprofil_f20_100_gray" model_filename="aluprofil_f20_100_gray.dae" scale="0.001"  size_x="0.02" size_y="0.02" size_z="0.1" weight="0.05"/>
 </robot>

File: mcr_environments/mcr_gazebo_objects/ros/urdf/aluprofil_s40_100_gray.urdf.xacro (robot description, xacro)
@@ -1,5 +1,5 @@
 <?xml version="1.0"?>
 <robot name="aluprofil_s40_100_gray" xmlns:xacro="http://ros.org/wiki/xacro">
-	<include filename="$(find mcr_gazebo_objects)/ros/templates/model.urdf.xacro" />
+	<xacro:include filename="$(find mcr_gazebo_objects)/ros/templates/model.urdf.xacro" />
 	<xacro:model_template name="aluprofil_s40_100_gray" model_filename="aluprofil_s40_100_gray.dae" scale="0.001"  size_x="0.04" size_y="0.04" size_z="0.1" weight="0.185"/>
 </robot>

File: mcr_environments/mcr_gazebo_objects/ros/urdf/bolt_m20_100.urdf.xacro (robot description, xacro)
@@ -1,5 +1,5 @@
 <?xml version="1.0"?>
 <robot name="bolt_m20_100" xmlns:xacro="http://ros.org/wiki/xacro">
-	<include filename="$(find mcr_gazebo_objects)/ros/templates/model.urdf.xacro" />
+	<xacro:include filename="$(find mcr_gazebo_objects)/ros/templates/model.urdf.xacro" />
 	<xacro:model_template name="bolt_m20_100" model_filename="bolt_m20_100.dae" scale="0.001"  size_x="0.11" size_y="0.02" size_z="0.02" weight="0.290"/>
 </robot>

File: mcr_environments/mcr_gazebo_objects/ros/urdf/bolt_m20_180.urdf.xacro (robot description, xacro)
@@ -1,5 +1,5 @@
 <?xml version="1.0"?>
 <robot name="bolt_m20_180" xmlns:xacro="http://ros.org/wiki/xacro">
-	<include filename="$(find mcr_gazebo_objects)/ros/templates/model.urdf.xacro" />
+	<xacro:include filename="$(find mcr_gazebo_objects)/ros/templates/model.urdf.xacro" />
 	<xacro:model_template name="bolt_m20_180" model_filename="bolt_m20_180.dae" scale="0.001"  size_x="0.11" size_y="0.02" size_z="0.02" weight="0.477"/>
 </robot>

File: mcr_environments/mcr_gazebo_objects/ros/urdf/nut_m20.urdf.xacro (robot description, xacro)
@@ -1,5 +1,5 @@
 <?xml version="1.0"?>
 <robot name="nut_m20" xmlns:xacro="http://ros.org/wiki/xacro">
-	<include filename="$(find mcr_gazebo_objects)/ros/templates/model.urdf.xacro" />
+	<xacro:include filename="$(find mcr_gazebo_objects)/ros/templates/model.urdf.xacro" />
 	<xacro:model_template name="nut_m20" model_filename="nut_m20.dae" scale="0.001"  size_x="0.015" size_y="0.028" size_z="0.028" weight="0.068"/>
 </robot>

File: mcr_environments/mcr_gazebo_objects/ros/urdf/nut_m30.urdf.xacro (robot description, xacro)
@@ -1,5 +1,5 @@
 <?xml version="1.0"?>
 <robot name="nut_m30" xmlns:xacro="http://ros.org/wiki/xacro">
-	<include filename="$(find mcr_gazebo_objects)/ros/templates/model.urdf.xacro" />
+	<xacro:include filename="$(find mcr_gazebo_objects)/ros/templates/model.urdf.xacro" />
 	<xacro:model_template name="nut_m30" model_filename="nut_m30.dae" scale="0.001"  size_x="0.025" size_y="0.045" size_z="0.045"  weight="0.215"/>
 </robot>

Commit message: remove entries which are already defined somewhere else

File: mcr_common/mcr_description/urdf/materials.urdf.xacro (robot description, xacro)
@@ -1,12 +1,6 @@
 <?xml version="1.0"?>
 <root>
-  <material name="Blue">
-    <color rgba="0.0 0.0 0.8 1.0"/>
-  </material>
   <material name="Grey2">
     <color rgba="0.9 0.9 0.9 1.0"/>
-  </material>
-  <material name="LightGrey">
-    <color rgba="0.82 0.82 0.82 1.0"/>
   </material>
   <material name="Caster">
