Commit message: Added convex hull of asus and scaled convex hull larger for collision
Generated convex hull of asus camera

In asus xacro:
- Include youbot_description asus_xtion_camera.gazebo.xacro
-- Because there is a bug in mcr_description version
- use new convex hull for collision geometry, scaling up by 1mm->2mm to avoid collisions with objects in gripper

File: mcr_common/mcr_description/urdf/sensors/asus_xtion_camera.urdf.xacro (robot description, xacro)
@@ -1,5 +1,5 @@
 <?xml version="1.0"?>
 <root xmlns:xacro="http://playerstage.sourceforge.net/gazebo/xmlschema/#interface">
-  <xacro:include filename="$(find mcr_description)/urdf/sensors/asus_xtion_camera.gazebo.xacro" />
+  <xacro:include filename="$(find youbot_description)/urdf/sensors/asus_xtion_camera.gazebo.xacro" />
   <property name="eye_x_offset" value="0.03" />
   <property name="eye_y_offset" value="0.035" />
@@ -88,5 +88,5 @@
         <origin xyz="0.02 -0.03 0" rpy="${M_PI/2} 0 ${M_PI/2}" />
         <geometry>
-           <mesh filename="package://mcr_description/meshes/sensors/asus_xtion_pro_live_camera.dae" scale="0.001 0.001 0.001"/>
+           <mesh filename="package://mcr_description/meshes/sensors/asus_xtion_pro_live_camera_convexhull.dae" scale="0.002 0.002 0.002"/>
         </geometry>
       </collision >

Commit message: reduced asus camera scale size in urdf

File: mcr_common/mcr_description/urdf/sensors/asus_xtion_camera.urdf.xacro (robot description, xacro)
@@ -88,5 +88,5 @@
         <origin xyz="0.02 -0.03 0" rpy="${M_PI/2} 0 ${M_PI/2}" />
         <geometry>
-           <mesh filename="package://mcr_description/meshes/sensors/asus_xtion_pro_live_camera_convexhull.dae" scale="0.002 0.002 0.002"/>
+           <mesh filename="package://mcr_description/meshes/sensors/asus_xtion_pro_live_camera_convexhull.dae" scale="0.001 0.001 0.001"/>
         </geometry>
       </collision >

Commit message: fix bug in ASUS Xtion urdf file

File: mcr_common/mcr_description/urdf/sensors/asus_xtion_camera.urdf.xacro (robot description, xacro)
@@ -65,5 +65,5 @@
       </collision >
     </link>
-    <joint name="asus_xtion_tilt_joint" type="fixed">
+    <joint name="${name}_tilt_joint" type="fixed">
      	<parent link="${name}_foot_link"/>
      	<child link="${name}_tilt_link"/>
