Commit message: Fixes model of realsense camera
The faces of the previous solid were flipped, causing collision detection
to fail.

- Regenerated fixed version of model.
- Adds convex hull version of model for collision checking.
- fixes unit scaling from inch to m ( 0.0254 )

File: mcr_common/mcr_description/urdf/sensors/realsense_camera.urdf.xacro (robot description, xacro)
@@ -5,5 +5,5 @@
        xmlns:xacro="http://ros.org/wiki/xacro">
   <xacro:macro name="realsense_camera" params="name parent *origin">
-  	<link name="${name}_link">
+    <link name="${name}_link">
       <inertial>
         <mass value="0.1" />
@@ -14,5 +14,5 @@
           <origin xyz="0 0 0" rpy="0 0 0" />
         <geometry>
-          <mesh filename="package://mcr_description/meshes/sensors/realsense_camera.dae" />
+          <mesh filename="package://mcr_description/meshes/sensors/realsense_camera.dae" scale="0.0254 0.0254 0.0254" />
         </geometry>
         <material name="LightGrey" />
@@ -21,5 +21,5 @@
         <origin xyz="0 0 0" rpy="0 0 0" />
         <geometry>
-          <mesh filename="package://mcr_description/meshes/sensors/realsense_camera.dae" />
+          <mesh filename="package://mcr_description/meshes/sensors/realsense_camera_convexhull.dae" scale="0.0254 0.0254 0.0254" />
         </geometry>
      </collision>
