Commit message: [description] update intel realsense URDF and mesh

File: mcr_common/mcr_description/urdf/sensors/intel_realsense_f200_camera.urdf.xacro (robot description, xacro)
@@ -4,5 +4,5 @@
        xmlns:interface="http://playerstage.sourceforge.net/gazebo/xmlschema/#interface"
        xmlns:xacro="http://ros.org/wiki/xacro">
-  <xacro:macro name="realsense_camera" params="name parent *origin">
+  <xacro:macro name="intel_realsense_f200_camera" params="name parent *origin">
     <link name="${name}_link">
       <inertial>
@@ -12,14 +12,13 @@
       </inertial>
       <visual>
-          <origin xyz="0 0 0" rpy="0 0 0" />
+        <origin xyz="0 0 0" rpy="0 0 0" />
         <geometry>
-          <mesh filename="package://mcr_description/meshes/sensors/realsense_camera.dae" scale="0.0254 0.0254 0.0254" />
+          <mesh filename="package://mcr_description/meshes/sensors/intel_realsense_f200_camera.dae" scale="0.001 0.001 0.001" />
         </geometry>
-        <material name="LightGrey" />
       </visual>
       <collision>
         <origin xyz="0 0 0" rpy="0 0 0" />
         <geometry>
-          <mesh filename="package://mcr_description/meshes/sensors/realsense_camera_convexhull.dae" scale="0.0254 0.0254 0.0254" />
+          <mesh filename="package://mcr_description/meshes/sensors/intel_realsense_f200_camera_convex_hull.dae" scale="0.001 0.001 0.001" />
         </geometry>
      </collision>

Commit message: [description] add gazebo configuration for IntelRealSense F200

File: mcr_common/mcr_description/urdf/sensors/intel_realsense_f200_camera.urdf.xacro (robot description, xacro)
@@ -4,4 +4,21 @@
        xmlns:interface="http://playerstage.sourceforge.net/gazebo/xmlschema/#interface"
        xmlns:xacro="http://ros.org/wiki/xacro">
+  <xacro:include filename="$(find mcr_description)/urdf/sensors/intel_realsense_f200_camera.gazebo.xacro" />
+  <property name="eye_x_offset" value="0.03" />
+  <property name="eye_y_offset" value="0.035" />
+  <xacro:macro name="intel_realsense_f200_eye" params="suffix parent *origin">
+	<link name="${parent}_${suffix}_frame">
+	  <inertial>
+		<mass value="0.01" />
+		<origin xyz="0 0 0" />
+		<inertia ixx="0.1" ixy="0" ixz="0" iyy="0.1" iyz="0" izz="0.1" />
+	  </inertial>
+	</link>
+	<joint name="${parent}_${suffix}_joint" type="fixed">
+	  <parent link="${parent}_link"/>
+	  <child link="${parent}_${suffix}_frame"/>
+	  <insert_block name="origin"/>
+	</joint>
+  </xacro:macro>
   <xacro:macro name="intel_realsense_f200_camera" params="name parent *origin">
     <link name="${name}_link">
@@ -29,4 +46,24 @@
       <child link="${name}_link"/>
     </joint>
-  </xacro:macro>
+    <xacro:intel_realsense_f200_eye suffix="depth" parent="${name}">
+	  <origin xyz="${eye_x_offset} ${eye_y_offset - 0.02} 0" rpy="0 0 0" />
+    </xacro:intel_realsense_f200_eye>
+    <xacro:intel_realsense_f200_eye suffix="depth_optical" parent="${name}">
+      <origin xyz="${eye_x_offset} ${eye_y_offset - 0.02} 0" rpy="${-M_PI/2} 0 ${-M_PI/2}" />
+    </xacro:intel_realsense_f200_eye>
+    <xacro:intel_realsense_f200_eye suffix="rgb" parent="${name}">
+      <origin xyz="${eye_x_offset} ${eye_y_offset - 0.04} 0" rpy="0 0 0" />
+    </xacro:intel_realsense_f200_eye>
+    <xacro:intel_realsense_f200_eye suffix="rgb_optical" parent="${name}">
+      <origin xyz="${eye_x_offset} ${eye_y_offset - 0.04} 0" rpy="${-M_PI/2} 0 ${-M_PI/2}" />
+    </xacro:intel_realsense_f200_eye>
+    <xacro:intel_realsense_f200_eye suffix="laser" parent="${name}">
+      <origin xyz="${eye_x_offset} ${eye_y_offset - 0.09} 0" rpy="0 0 0" />
+    </xacro:intel_realsense_f200_eye>
+    <xacro:intel_realsense_f200_eye suffix="laser_optical" parent="${name}">
+      <origin xyz="${eye_x_offset} ${eye_y_offset - 0.09} 0" rpy="${M_PI/2} 0 ${-M_PI/2}" />
+    </xacro:intel_realsense_f200_eye>
+     <!-- for simulation -->
+     <xacro:intel_realsense_f200_camera_gazebo name="${name}" />
+   </xacro:macro>
 </root>

Commit message: [description] fix realsense calibration

File: mcr_common/mcr_description/urdf/sensors/intel_realsense_f200_camera.urdf.xacro (robot description, xacro)
@@ -5,6 +5,7 @@
        xmlns:xacro="http://ros.org/wiki/xacro">
   <xacro:include filename="$(find mcr_description)/urdf/sensors/intel_realsense_f200_camera.gazebo.xacro" />
-  <property name="eye_x_offset" value="0.03" />
-  <property name="eye_y_offset" value="0.035" />
+  <property name="eye_x_offset" value="-0.015" />
+  <property name="eye_y_offset" value="0.024" />
+  <property name="eye_z_offset" value="0.018" />
   <xacro:macro name="intel_realsense_f200_eye" params="suffix parent *origin">
 	<link name="${parent}_${suffix}_frame">
@@ -29,5 +30,5 @@
       </inertial>
       <visual>
-        <origin xyz="0 0 0" rpy="0 0 0" />
+        <origin xyz="0 -0.074 0" rpy="0 0 0" />
         <geometry>
           <mesh filename="package://mcr_description/meshes/sensors/intel_realsense_f200_camera.dae" scale="0.001 0.001 0.001" />
@@ -35,5 +36,5 @@
       </visual>
       <collision>
-        <origin xyz="0 0 0" rpy="0 0 0" />
+        <origin xyz="0 -0.074 0" rpy="0 0 0" />
         <geometry>
           <mesh filename="package://mcr_description/meshes/sensors/intel_realsense_f200_camera_convex_hull.dae" scale="0.001 0.001 0.001" />
@@ -47,20 +48,20 @@
     </joint>
     <xacro:intel_realsense_f200_eye suffix="depth" parent="${name}">
-	  <origin xyz="${eye_x_offset} ${eye_y_offset - 0.02} 0" rpy="0 0 0" />
+      <origin xyz="${eye_x_offset} ${eye_y_offset - 0.048} ${eye_z_offset}" rpy="0 0 0" />
     </xacro:intel_realsense_f200_eye>
     <xacro:intel_realsense_f200_eye suffix="depth_optical" parent="${name}">
-      <origin xyz="${eye_x_offset} ${eye_y_offset - 0.02} 0" rpy="${-M_PI/2} 0 ${-M_PI/2}" />
+      <origin xyz="${eye_x_offset} ${eye_y_offset - 0.048} ${eye_z_offset}" rpy="${-M_PI/2} 0 ${-M_PI/2}" />
     </xacro:intel_realsense_f200_eye>
     <xacro:intel_realsense_f200_eye suffix="rgb" parent="${name}">
-      <origin xyz="${eye_x_offset} ${eye_y_offset - 0.04} 0" rpy="0 0 0" />
+      <origin xyz="${eye_x_offset} ${eye_y_offset - 0.024} ${eye_z_offset}" rpy="0 0 0" />
     </xacro:intel_realsense_f200_eye>
     <xacro:intel_realsense_f200_eye suffix="rgb_optical" parent="${name}">
-      <origin xyz="${eye_x_offset} ${eye_y_offset - 0.04} 0" rpy="${-M_PI/2} 0 ${-M_PI/2}" />
+      <origin xyz="${eye_x_offset} ${eye_y_offset - 0.024} ${eye_z_offset}" rpy="${-M_PI/2} 0 ${-M_PI/2}" />
     </xacro:intel_realsense_f200_eye>
     <xacro:intel_realsense_f200_eye suffix="laser" parent="${name}">
-      <origin xyz="${eye_x_offset} ${eye_y_offset - 0.09} 0" rpy="0 0 0" />
+      <origin xyz="${eye_x_offset} ${eye_y_offset} ${eye_z_offset}" rpy="0 0 0" />
     </xacro:intel_realsense_f200_eye>
     <xacro:intel_realsense_f200_eye suffix="laser_optical" parent="${name}">
-      <origin xyz="${eye_x_offset} ${eye_y_offset - 0.09} 0" rpy="${M_PI/2} 0 ${-M_PI/2}" />
+      <origin xyz="${eye_x_offset} ${eye_y_offset} ${eye_z_offset}" rpy="${M_PI/2} 0 ${-M_PI/2}" />
     </xacro:intel_realsense_f200_eye>
      <!-- for simulation -->
