Commit message: Added parameters and noise to the gazebo plugin

File: mcr_common/mcr_description/urdf/sensors/realsense_d435.gazebo.xacro (robot description, xacro)
@@ -4,9 +4,9 @@
       xmlns:interface="http://playerstage.sourceforge.net/gazebo/xmlschema/#interface"
       xmlns:xacro="http://ros.org/wiki/xacro">
-  <xacro:macro name="realsense_d435_gazebo">
-      <gazebo reference="camera_link">
-        <sensor type="depth" name="depth_sensor">
+  <xacro:macro name="realsense_d435_gazebo" params="name color:=rgb">
+      <gazebo reference="${name}_camera_link">
+        <sensor type="depth" name="${name}_depth_sensor">
           <update_rate>30.0</update_rate>
-          <camera name="camera_name">
+          <camera name="${name}_camera">
             <horizontal_fov>1.588</horizontal_fov>
             <image>
@@ -19,16 +19,21 @@
               <far>30.0</far>
             </clip>
+            <noise>
+              <type>gaussian</type>
+              <mean>0.0</mean>
+              <stddev>0.007</stddev>
+            </noise>
           </camera>
-          <plugin name="depth_sensor_plugin" filename="libgazebo_ros_openni_kinect.so">
+          <plugin name="${name}_realsense_d435_plugin" filename="libgazebo_ros_openni_kinect.so">
             <baseline>0.2</baseline>
             <alwaysOn>true</alwaysOn>
             <updateRate>0.0</updateRate>
-            <cameraName>camera_ir</cameraName>
-            <imageTopicName>/camera/color/image_raw</imageTopicName>
-            <cameraInfoTopicName>/camera/color/camera_info</cameraInfoTopicName>
-            <depthImageTopicName>/camera/depth/image_raw</depthImageTopicName>
-            <depthImageInfoTopicName>/camera/depth/camera_info</depthImageInfoTopicName>
-            <pointCloudTopicName>/camera/depth/points</pointCloudTopicName>
-            <frameName>/camera_link_optical</frameName>
+            <cameraName>${name}_ir</cameraName>
+            <imageTopicName>/${name}/${color}/image_raw</imageTopicName>
+            <cameraInfoTopicName>/${name}/${color}/camera_info</cameraInfoTopicName>
+            <depthImageTopicName>/${name}/depth/image_raw</depthImageTopicName>
+            <depthImageInfoTopicName>/${name}/depth/camera_info</depthImageInfoTopicName>
+            <pointCloudTopicName>/${name}/depth_registered/points</pointCloudTopicName>
+            <frameName>/${name}_camera_link_optical</frameName>
             <pointCloudCutoff>0.105</pointCloudCutoff>
             <pointCloudCutoffMax>10.0</pointCloudCutoffMax>

File: mcr_common/mcr_description/urdf/sensors/realsense_d435.urdf.xacro (robot description, xacro)
@@ -10,10 +10,10 @@
       <color rgba="0.5 0.5 0.5 1"/>
     </material>
-    <joint name="camera_link_joint" type="fixed">
+    <joint name="${name}_camera_link_joint" type="fixed">
       <xacro:insert_block name="origin" />
       <parent link="${parent}"/>
-      <child link="camera_link" />
+      <child link="${name}_camera_link" />
     </joint>
-    <link name="camera_link">
+    <link name="${name}_camera_link">
       <visual>
         <origin xyz="0.0149 -0.0175 0" rpy="${M_PI/2} 0 ${M_PI/2}"/>
@@ -35,11 +35,11 @@
       </inertial>
     </link>
-    <joint name="camera_link_optical_joint" type="fixed">
+    <joint name="${name}_camera_link_optical_joint" type="fixed">
       <origin xyz="0.0 0.0 0.0" rpy="${-M_PI/2} 0.0 ${-M_PI/2}" />
-      <parent link="camera_link"/>
-      <child link="camera_link_optical" />
+      <parent link="${name}_camera_link"/>
+      <child link="${name}_camera_link_optical" />
     </joint>
-    <link name="camera_link_optical" />
-    <xacro:realsense_d435_gazebo />
+    <link name="${name}_camera_link_optical" />
+    <xacro:realsense_d435_gazebo name="${name}" />
   </xacro:macro>
 </root>

Commit message: Used complete urdf description from realsense_description repository

File: mcr_common/mcr_description/urdf/sensors/realsense_d435.gazebo.xacro (robot description, xacro)
@@ -35,5 +35,5 @@
             <depthImageInfoTopicName>/${name}/depth/camera_info</depthImageInfoTopicName>
             <pointCloudTopicName>/${name}/depth_registered/points</pointCloudTopicName>
-            <frameName>/${name}_camera_link_optical</frameName>
+            <frameName>/${name}_camera_depth_optical_frame</frameName>
             <pointCloudCutoff>0.105</pointCloudCutoff>
             <pointCloudCutoffMax>10.0</pointCloudCutoffMax>

File: mcr_common/mcr_description/urdf/sensors/realsense_d435.urdf.xacro (robot description, xacro)
@@ -1,14 +1,35 @@
 <?xml version="1.0"?>
-<root xmlns:sensor="http://playerstage.sourceforge.net/gazebo/xmlschema/#sensor"
-       xmlns:controller="http://playerstage.sourceforge.net/gazebo/xmlschema/#controller"
-       xmlns:interface="http://playerstage.sourceforge.net/gazebo/xmlschema/#interface"
-       xmlns:xacro="http://ros.org/wiki/xacro">
+<!--
+License: Apache 2.0. See LICENSE file in root directory.
+Copyright(c) 2017 Intel Corporation. All Rights Reserved
+This is the URDF model for the Intel RealSense 430 camera, in it's
+aluminum peripherial evaluation case.
+-->
+<robot xmlns:xacro="http://ros.org/wiki/xacro">
   <xacro:include filename="$(find mcr_description)/urdf/sensors/realsense_d435.gazebo.xacro" />
   <xacro:macro name="realsense_d435" params="name parent *origin">
     <xacro:property name="M_PI" value="3.1415926535897931" />
-    <material name="aluminum">
-      <color rgba="0.5 0.5 0.5 1"/>
+    <!-- The following values are approximate, and the camera node
+     publishing TF values with actual calibrated camera extrinsic values -->
+    <xacro:property name="d435_cam_depth_to_left_ir_offset" value="0.0"/>
+    <xacro:property name="d435_cam_depth_to_right_ir_offset" value="-0.050"/>
+    <xacro:property name="d435_cam_depth_to_color_offset" value="0.015"/>
+    <!-- The following values model the aluminum peripherial case for the
+  	D435 camera, with the camera joint represented by the actual
+  	peripherial camera tripod mount -->
+    <xacro:property name="d435_cam_width" value="0.090"/>
+    <xacro:property name="d435_cam_height" value="0.025"/>
+    <xacro:property name="d435_cam_depth" value="0.02505"/>
+    <xacro:property name="d435_cam_mount_from_center_offset" value="0.0149"/>
+    <!-- The following offset is relative the the physical D435 camera peripherial
+  	camera tripod mount -->
+    <xacro:property name="d435_cam_depth_px" value="${d435_cam_mount_from_center_offset}"/>
+    <xacro:property name="d435_cam_depth_py" value="0.0175"/>
+    <xacro:property name="d435_cam_depth_pz" value="${d435_cam_height/2}"/>
+    <material name="${name}_aluminum">
+	  <color rgba="0.5 0.5 0.5 1"/>
     </material>
-    <joint name="${name}_camera_link_joint" type="fixed">
+    <!-- camera body, with origin at bottom screw mount -->
+    <joint name="${name}_camera_joint" type="fixed">
       <xacro:insert_block name="origin" />
       <parent link="${parent}"/>
@@ -17,17 +38,18 @@
     <link name="${name}_camera_link">
       <visual>
-        <origin xyz="0.0149 -0.0175 0" rpy="${M_PI/2} 0 ${M_PI/2}"/>
+      <origin xyz="${d435_cam_mount_from_center_offset} 0.0 ${d435_cam_height/2}" rpy="${M_PI/2} 0 ${M_PI/2}"/>
         <geometry>
-            <mesh filename="package://mcr_description/meshes/sensors/realsense_d435.dae" />
+          <mesh filename="package://mcr_description/meshes/sensors/realsense_d435.dae" />
         </geometry>
-        <material name="aluminum"/>
+        <material name="${name}_aluminum"/>
       </visual>
       <collision>
-        <origin xyz="0 -0.0175 0" rpy="0 0 0"/>
+        <origin xyz="0.0 0.0 ${d435_cam_height/2}" rpy="0 0 0"/>
         <geometry>
-        <box size="0.02505 0.09 0.025"/>
+        <box size="${d435_cam_depth} ${d435_cam_width} ${d435_cam_height}"/>
         </geometry>
       </collision>
       <inertial>
+        <!-- The following are not reliable values, and should not be used for modeling -->
         <mass value="0.564" />
         <origin xyz="0 0 0" />
@@ -35,11 +57,57 @@
       </inertial>
     </link>
-    <joint name="${name}_camera_link_optical_joint" type="fixed">
-      <origin xyz="0.0 0.0 0.0" rpy="${-M_PI/2} 0.0 ${-M_PI/2}" />
+    <!-- camera depth joints and links -->
+    <joint name="${name}_camera_depth_joint" type="fixed">
+      <origin xyz="${d435_cam_depth_px} ${d435_cam_depth_py} ${d435_cam_depth_pz}" rpy="0 0 0"/>
       <parent link="${name}_camera_link"/>
-      <child link="${name}_camera_link_optical" />
+      <child link="${name}_camera_depth_frame" />
     </joint>
-    <link name="${name}_camera_link_optical" />
+    <link name="${name}_camera_depth_frame"/>
+    <joint name="${name}_camera_depth_optical_joint" type="fixed">
+      <origin xyz="0 0 0" rpy="${-M_PI/2} 0 ${-M_PI/2}" />
+      <parent link="${name}_camera_depth_frame" />
+      <child link="${name}_camera_depth_optical_frame" />
+    </joint>
+    <link name="${name}_camera_depth_optical_frame"/>
+    <!-- camera left IR joints and links -->
+    <joint name="${name}_camera_left_ir_joint" type="fixed">
+      <origin xyz="0 ${d435_cam_depth_to_left_ir_offset} 0" rpy="0 0 0" />
+      <parent link="${name}_camera_depth_frame" />
+      <child link="${name}_camera_left_ir_frame" />
+    </joint>
+    <link name="${name}_camera_left_ir_frame"/>
+    <joint name="${name}_camera_left_ir_optical_joint" type="fixed">
+      <origin xyz="0 0 0" rpy="${-M_PI/2} 0 ${-M_PI/2}" />
+      <parent link="${name}_camera_left_ir_frame" />
+      <child link="${name}_camera_left_ir_optical_frame" />
+    </joint>
+    <link name="${name}_camera_left_ir_optical_frame"/>
+    <!-- camera right IR joints and links -->
+    <joint name="${name}_camera_right_ir_joint" type="fixed">
+      <origin xyz="0 ${d435_cam_depth_to_right_ir_offset} 0" rpy="0 0 0" />
+      <parent link="${name}_camera_depth_frame" />
+      <child link="${name}_camera_right_ir_frame" />
+    </joint>
+    <link name="${name}_camera_right_ir_frame"/>
+    <joint name="${name}_camera_right_ir_optical_joint" type="fixed">
+      <origin xyz="0 0 0" rpy="${-M_PI/2} 0 ${-M_PI/2}" />
+      <parent link="${name}_camera_right_ir_frame" />
+      <child link="${name}_camera_right_ir_optical_frame" />
+    </joint>
+    <link name="${name}_camera_right_ir_optical_frame"/>
+    <!-- camera color joints and links -->
+    <joint name="${name}_camera_color_joint" type="fixed">
+      <origin xyz="0 ${d435_cam_depth_to_color_offset} 0" rpy="0 0 0" />
+      <parent link="${name}_camera_depth_frame" />
+      <child link="${name}_camera_color_frame" />
+    </joint>
+    <link name="${name}_camera_color_frame"/>
+    <joint name="${name}_camera_color_optical_joint" type="fixed">
+      <origin xyz="0 0 0" rpy="${-M_PI/2} 0 ${-M_PI/2}" />
+      <parent link="${name}_camera_color_frame" />
+      <child link="${name}_camera_color_optical_frame" />
+    </joint>
+    <link name="${name}_camera_color_optical_frame"/>
     <xacro:realsense_d435_gazebo name="${name}" />
   </xacro:macro>
-</root>
+</robot>
