Commit message: Adds simple convex hull of microsoft mount for collision checking
- Convex hull created using MeshLab.
- Modified xacro to use convex hull for collision geometry.

Notes:
- rendering appears odd because the mesh is not watertight, but all points are present.
- mount model is static forward facing, so it doesn't account for the rotation set with the bevel gears. which changes the collision geometry slightly, but would require much more work, I will look into it when I make the festo non static.

Moved cam mount from sensors dir to mounts dir

- Created mounts subdirectories and moved files

File: mcr_common/mcr_description/urdf/mounts/microsoft_lifecam_1080_mount.urdf.xacro (robot description, xacro)
@@ -14,5 +14,5 @@
         <origin xyz="-0.015 0.04 -0.055" rpy="0 0 -1.57079633" />
         <geometry>
-          <mesh filename="package://mcr_description/meshes/sensors/microsoft_lifecam_1080_mount.dae" scale="0.001 0.001 0.001" />
+          <mesh filename="package://mcr_description/meshes/mounts/microsoft_lifecam_1080_mount.dae" scale="0.001 0.001 0.001" />
         </geometry>
         <material name="Black" />
@@ -21,5 +21,5 @@
         <origin xyz="-0.015 0.04 -0.055" rpy="0 0 -1.57079633" />
         <geometry>
-          <mesh filename="package://mcr_description/meshes/sensors/microsoft_lifecam_1080_mount.dae" scale="0.001 0.001 0.001"/>
+          <mesh filename="package://mcr_description/meshes/mounts/microsoft_lifecam_1080_mount_convexhull.dae" scale="0.001 0.001 0.001"/>
         </geometry>
       </collision >
