Commit message: [description] fix dynamixel motor URDF

File: mcr_common/mcr_description/urdf/motors/dynamixel_motor_ax-12a.urdf.xacro (robot description, xacro)
@@ -4,9 +4,37 @@
        xmlns:interface="http://playerstage.sourceforge.net/gazebo/xmlschema/#interface"
        xmlns:xacro="http://ros.org/wiki/xacro">
+  <xacro:include filename="$(find mcr_description)/urdf/motors/dynamixel_motor_ax-12a.gazebo.xacro" />
+  <xacro:include filename="$(find mcr_description)/urdf/motors/dynamixel_motor_ax-12a.transmission.xacro" />
   <xacro:macro name="dynamixel_motor_AX-12A" params="parent name *origin">
-    <joint name="${name}_joint" type="fixed" >
+    <joint name="${name}_base_joint" type="fixed" >
       <insert_block name="origin" />
       <parent link="${parent}" />
+      <child link="${name}_base_link" />
+    </joint>
+    <link name="${name}_base_link">
+      <inertial>
+        <origin xyz="0 0 0" rpy="0 0 0"/>
+        <mass value="0.01"/>
+        <inertia ixx="0.01" ixy="0" ixz="0" iyy="0.01" iyz="0" izz="0.01" />
+      </inertial>
+      <visual>
+        <origin xyz="0 0 0.03" rpy="0 ${M_PI/2} 0" />
+        <geometry>
+          <mesh filename="package://mcr_description/meshes/motors/dynamixel_motor_ax-12a.dae" scale="0.001 0.001 0.001" />
+        </geometry>
+      </visual>
+      <collision>
+        <origin xyz="0 0 0.03" rpy="0 ${M_PI/2} 0" />
+        <geometry>
+          <mesh filename="package://mcr_description/meshes/motors/dynamixel_motor_ax-12a_convex_hull.dae" scale="0.001 0.001 0.001" />
+        </geometry>
+      </collision>
+    </link>
+    <joint name="${name}_joint" type="revolute" >
+      <parent link="${name}_base_link" />
       <child link="${name}_link" />
+      <origin xyz="0 0 0.03" rpy="0 0 0"/>
+      <axis xyz="-1 0 0"/>
+      <limit effort="1.5" lower="-${M_PI / 180 * 150}" upper="${M_PI / 180 * 150}" velocity="6.178465545"/>
     </joint>
     <link name="${name}_link">
@@ -16,17 +44,8 @@
         <inertia ixx="0.01" ixy="0" ixz="0" iyy="0.01" iyz="0" izz="0.01" />
       </inertial>
-      <visual>
-        <origin xyz="0 0 0" rpy="0 ${M_PI/2} 0" />
-        <geometry>
-          <mesh filename="package://mcr_description/meshes/motors/dynamixel_motor_ax-12a.dae" scale="0.001 0.001 0.001" />
-        </geometry>
-      </visual>
-      <collision>
-        <origin xyz="0 0 0" rpy="0 ${M_PI/2} 0" />
-        <geometry>
-          <mesh filename="package://mcr_description/meshes/motors/dynamixel_motor_ax-12a_convex_hull.dae" scale="0.001 0.001 0.001" />
-        </geometry>
-      </collision>
     </link>
+    <!-- extensions -->
+	<xacro:dynamixel_motor_AX-12A_gazebo name="${name}" />
+	<xacro:dynamixel_motor_AX-12A_transmission name="${name}" />
   </xacro:macro>
 </robot>

Commit message: [description] add motor direction parameter for dynamixel URDF

File: mcr_common/mcr_description/urdf/motors/dynamixel_motor_ax-12a.urdf.xacro (robot description, xacro)
@@ -6,5 +6,5 @@
   <xacro:include filename="$(find mcr_description)/urdf/motors/dynamixel_motor_ax-12a.gazebo.xacro" />
   <xacro:include filename="$(find mcr_description)/urdf/motors/dynamixel_motor_ax-12a.transmission.xacro" />
-  <xacro:macro name="dynamixel_motor_AX-12A" params="parent name *origin">
+  <xacro:macro name="dynamixel_motor_AX-12A" params="parent name *origin motor_direction">
     <joint name="${name}_base_joint" type="fixed" >
       <insert_block name="origin" />
@@ -34,6 +34,6 @@
       <parent link="${name}_base_link" />
       <child link="${name}_link" />
-      <origin xyz="0 0 0.03" rpy="0 0 0"/>
-      <axis xyz="-1 0 0"/>
+      <origin xyz="0 0 0.03" rpy="0 0 ${M_PI}"/>
+      <axis xyz="${motor_direction} 0 0"/>
       <limit effort="1.5" lower="-${M_PI / 180 * 150}" upper="${M_PI / 180 * 150}" velocity="6.178465545"/>
     </joint>

Commit message: [description] use param to set position offset

File: mcr_common/mcr_description/urdf/motors/dynamixel_motor_ax-12a.urdf.xacro (robot description, xacro)
@@ -6,5 +6,5 @@
   <xacro:include filename="$(find mcr_description)/urdf/motors/dynamixel_motor_ax-12a.gazebo.xacro" />
   <xacro:include filename="$(find mcr_description)/urdf/motors/dynamixel_motor_ax-12a.transmission.xacro" />
-  <xacro:macro name="dynamixel_motor_AX-12A" params="parent name *origin motor_direction">
+  <xacro:macro name="dynamixel_motor_AX-12A" params="parent name *origin motor_direction position_offset">
     <joint name="${name}_base_joint" type="fixed" >
       <insert_block name="origin" />
@@ -34,5 +34,5 @@
       <parent link="${name}_base_link" />
       <child link="${name}_link" />
-      <origin xyz="0 0 0.03" rpy="0 0 ${M_PI}"/>
+      <origin xyz="0 0 0.03" rpy="${position_offset} 0 ${M_PI}"/>
       <axis xyz="${motor_direction} 0 0"/>
       <limit effort="1.5" lower="-${M_PI / 180 * 150}" upper="${M_PI / 180 * 150}" velocity="6.178465545"/>
