Commit message: [description] fix masses temporally
to get the arm properly working in simulation

File: mcr_common/mcr_description/urdf/motors/dynamixel_bracket_fp04-f2.urdf.xacro (robot description, xacro)
@@ -13,5 +13,5 @@
       <inertial>
         <origin xyz="0 0 0" rpy="0 0 0"/>
-        <mass value="0.1"/>
+        <mass value="0.001"/>
         <inertia ixx="0.01" ixy="0" ixz="0" iyy="0.01" iyz="0" izz="0.01" />
       </inertial>

File: mcr_common/mcr_description/urdf/motors/dynamixel_motor_ax-12a.urdf.xacro (robot description, xacro)
@@ -41,5 +41,5 @@
       <inertial>
         <origin xyz="0 0 0" rpy="0 0 0"/>
-        <mass value="0.1"/>
+        <mass value="0.001"/>
         <inertia ixx="0.01" ixy="0" ixz="0" iyy="0.01" iyz="0" izz="0.01" />
       </inertial>

Commit message: [mcr_description] updated dynamixel masses

File: mcr_common/mcr_description/urdf/motors/dynamixel_bracket_fp04-f2.urdf.xacro (robot description, xacro)
@@ -13,5 +13,5 @@
       <inertial>
         <origin xyz="0 0 0" rpy="0 0 0"/>
-        <mass value="0.001"/>
+        <mass value="0.011"/>
         <inertia ixx="0.01" ixy="0" ixz="0" iyy="0.01" iyz="0" izz="0.01" />
       </inertial>

File: mcr_common/mcr_description/urdf/motors/dynamixel_motor_ax-12a.urdf.xacro (robot description, xacro)
@@ -15,5 +15,5 @@
       <inertial>
         <origin xyz="0 0 0" rpy="0 0 0"/>
-        <mass value="0.01"/>
+        <mass value="0.054"/>
         <inertia ixx="0.01" ixy="0" ixz="0" iyy="0.01" iyz="0" izz="0.01" />
       </inertial>
