Commit message: [mcr_gazebo_worlds] The brsu-c069 world urdf was causing Gazebo to crash on kinetic

File: mcr_environments/mcr_gazebo_worlds/common/worlds/brsu-c069.urdf.xacro (robot description, xacro)
@@ -18,11 +18,11 @@
 			<origin xyz="0 0 0" />
 			<geometry>
-				<box size="0.00 0.00 0.00" />
-			</geometry>
-		</visual>
-		<collision>
-			<origin xyz="0 0 0" />
-			<geometry>
-				<box size="0.00 0.00 0.00" />
+				<box size="0.01 0.01 0.01" />
+			</geometry>
+		</visual>
+		<collision>
+			<origin xyz="0 0 0" />
+			<geometry>
+				<box size="0.01 0.01 0.01" />
 			</geometry>
 		</collision>
