Commit message: geometry values in the map are changed to a non-zero value. (Gazebo7 and gazebo9 is buggy, size=0 values are taken as NaN)

File: mcr_environments/mcr_gazebo_worlds/common/worlds/brsu-c025-sim.urdf.xacro (robot description, xacro)
@@ -31,11 +31,11 @@
       			<origin xyz="0 0 0" />
       			<geometry>
-					<box size="0 0 0" />
-      			</geometry>
-    		</visual>
-			<collision>
-      			<origin xyz="0 0 0"/>
-				<geometry>
-					<box size="0 0 0"/>
+					<box size="0.01 0.01 0.01" />
+      			</geometry>
+    		</visual>
+			<collision>
+      			<origin xyz="0 0 0"/>
+				<geometry>
+					<box size="0.01 0.01 0.01"/>
 				</geometry>
     		</collision>
@@ -128,5 +128,5 @@
       			<origin xyz="0 0 0"/>
       			<geometry>
-					<box size="0 0 0" /> <!--Insert 120 wall here for closed arena-->
+					<box size="0.01 0.01 0.01" /> <!--Insert 120 wall here for closed arena-->
 					<!--box size="0.04 1.2 0.3" /--> <!--wall 120, width = 4 cm, lenght = 120 cm, height = 30 cm-->
       			</geometry>
@@ -135,5 +135,5 @@
       			<origin xyz="0 0 0"/>
 				<geometry>
-					<box size="0 0 0" /> <!--Insert 120 wall here for closed arena-->
+					<box size="0.01 0.01 0.01" /> <!--Insert 120 wall here for closed arena-->
 					<!--box size="0.04 0.8 0.3"/-->
 				</geometry>
@@ -155,5 +155,5 @@
       			<origin xyz="0 0 0"/>
       			<geometry>
-					<box size="0 0 0" /> <!--Insert 80 wall here for closed arena-->
+					<box size="0.01 0.01 0.01" /> <!--Insert 80 wall here for closed arena-->
 					<!--box size="0.04 0.8 0.3" /--> <!--wall 80, width = 4 cm, lenght = 80 cm, height = 30 cm-->
       			</geometry>
@@ -162,5 +162,5 @@
       			<origin xyz="0 0 0"/>
 				<geometry>
-					<box size="0 0 0" /> <!--Insert 80 wall here for closed arena-->
+					<box size="0.01 0.01 0.01" /> <!--Insert 80 wall here for closed arena-->
 					<!--box size="0.04 0.8 0.3"/-->
 				</geometry>
@@ -302,5 +302,5 @@
       			<origin xyz="0 0 0"/>
       			<geometry>
-					<box size="0 0 0" /> <!--Insert 120 wall here for closed arena-->
+					<box size="0.01 0.01 0.01" /> <!--Insert 120 wall here for closed arena-->
 					<!--box size="0.04 1.2 0.3" /--> <!--wall 120, width = 4 cm, lenght = 120 cm, height = 30 cm-->
       			</geometry>
@@ -309,5 +309,5 @@
       			<origin xyz="0 0 0"/>
 				<geometry>
-					<box size="0 0 0" /> <!--Insert 120 wall here for closed arena-->
+					<box size="0.01 0.01 0.01" /> <!--Insert 120 wall here for closed arena-->
 					<!--box size="0.04 0.8 0.3"/-->
 				</geometry>
@@ -329,5 +329,5 @@
       			<origin xyz="0 0 0"/>
       			<geometry>
-					<box size="0 0 0" /> <!--Insert 80 wall here for closed arena-->
+					<box size="0.01 0.01 0.01" /> <!--Insert 80 wall here for closed arena-->
 					<!--box size="0.04 0.8 0.3" /--> <!--wall 80, width = 4 cm, lenght = 80 cm, height = 30 cm-->
       			</geometry>
@@ -336,5 +336,5 @@
       			<origin xyz="0 0 0"/>
 				<geometry>
-					<box size="0 0 0" /> <!--Insert 80 wall here for closed arena-->
+					<box size="0.01 0.01 0.01" /> <!--Insert 80 wall here for closed arena-->
 					<!--box size="0.04 0.8 0.3"/-->
 				</geometry>

Commit message: [simulation] Fixed floating walls in c025 gazebo world

File: mcr_environments/mcr_gazebo_worlds/common/worlds/brsu-c025-sim.urdf.xacro (robot description, xacro)
@@ -132,11 +132,11 @@
       			</geometry>
     		</visual>
-			<collision>
-      			<origin xyz="0 0 0"/>
-				<geometry>
-					<box size="0.01 0.01 0.01" /> <!--Insert 120 wall here for closed arena-->
-					<!--box size="0.04 0.8 0.3"/-->
-				</geometry>
-    		</collision>
+            <!-- Uncomment following block for closed arena -->
+			<!-- <collision> -->
+            <!-- <origin xyz="0 0 0"/> -->
+			<!-- 	<geometry> -->
+			<!-- 		<box size="0.04 0.8 0.3"/> -->
+			<!-- 	</geometry> -->
+    		<!-- </collision> -->
   	</link>
   	<joint name="join5" type="fixed">
@@ -159,11 +159,11 @@
       			</geometry>
     		</visual>
-			<collision>
-      			<origin xyz="0 0 0"/>
-				<geometry>
-					<box size="0.01 0.01 0.01" /> <!--Insert 80 wall here for closed arena-->
-					<!--box size="0.04 0.8 0.3"/-->
-				</geometry>
-    		</collision>
+            <!-- Uncomment following block for closed arena -->
+			<!-- <collision> -->
+            <!-- <origin xyz="0 0 0"/> -->
+			<!-- 	<geometry> -->
+			<!-- 		<box size="0.04 0.8 0.3"/> -->
+			<!-- 	</geometry> -->
+    		<!-- </collision> -->
   	</link>
   	<joint name="join6" type="fixed">
@@ -306,11 +306,11 @@
       			</geometry>
     		</visual>
-			<collision>
-      			<origin xyz="0 0 0"/>
-				<geometry>
-					<box size="0.01 0.01 0.01" /> <!--Insert 120 wall here for closed arena-->
-					<!--box size="0.04 0.8 0.3"/-->
-				</geometry>
-    		</collision>
+            <!-- Uncomment following block for closed arena -->
+			<!-- <collision> -->
+            <!-- <origin xyz="0 0 0"/> -->
+			<!-- 	<geometry> -->
+			<!-- 		<box size="0.04 0.8 0.3"/> -->
+			<!-- 	</geometry> -->
+    		<!-- </collision> -->
   	</link>
   	<joint name="join12" type="fixed">
@@ -333,11 +333,11 @@
       			</geometry>
     		</visual>
-			<collision>
-      			<origin xyz="0 0 0"/>
-				<geometry>
-					<box size="0.01 0.01 0.01" /> <!--Insert 80 wall here for closed arena-->
-					<!--box size="0.04 0.8 0.3"/-->
-				</geometry>
-    		</collision>
+            <!-- Uncomment following block for closed arena -->
+			<!-- <collision> -->
+            <!-- <origin xyz="0 0 0"/> -->
+			<!-- 	<geometry> -->
+			<!-- 		<box size="0.04 0.8 0.3"/> -->
+			<!-- 	</geometry> -->
+    		<!-- </collision> -->
   	</link>
   	<joint name="join13" type="fixed">

Commit message: [gazebo][world] Using ws, shelf and ppt models in c025 environment

File: mcr_environments/mcr_gazebo_worlds/common/worlds/brsu-c025-sim.urdf.xacro (robot description, xacro)
@@ -1,699 +1,264 @@
 <?xml version="1.0"?>
 <!--
-			brsu c025 lab configuration #2
-			Author: Oscar Lima
-			walls:
-				   7  _6___    5      4   _____3_
-					||8  |                  |17 || 2
-					||___|     _______    19|___||
-					          |22 |23 |     |16 || 1
-					  ___     |___|___|   20|___||
-					||15 |       21         |18 || 9
-					||___|_               __|___||
-				   14  13      12     11      10
-			tree:
-					1-2-3-4-5-6-7
-					6-8
-					1-9-10-11-12-13-14
-					13-15
-					1-16-17-18
-					1-19-20
-					1-21-22-23
+Name: brsu-c025-sim
+Author: Dharmin B.
+         _____________wall_3_____________
+        |          |          |          |
+        |   SH01   |   PP01   |   SH02   |
+        |__________|__________|__________|
+        |                                |
+        |                                |
+        |                                |
+        |                                |                ^ X
+        |           __________           |                |
+        |          |          |          |                |
+        |          |   WS04   |          |          <_____|
+        |          |__________|          |          Y
+   wall_2          |__wall_6__|          wall_4
+        |          |          |          |
+        |          |   WS03   |          |
+        |          |__________|          |
+        |                                |
+        |                                |
+        |                                |
+        |                                |
+        |__________            __________|
+        |          |          |          |
+        |   WS01   |  ORIGIN  |   WS02   |
+        |__________|          |__________|
+           wall_1                wall_5
 -->
-<robot name="brsu-c025-config2">
-  	<link name="origin">
-    		<inertial>
-      			<origin xyz="0 0 0" />
-      			<mass value="0" />
-      			<inertia  ixx="0" ixy="0"  ixz="0"  iyy="0"  iyz="0"  izz="0" />
-    		</inertial>
-    		<visual>
-      			<origin xyz="0 0 0" />
-      			<geometry>
-					<box size="0.01 0.01 0.01" />
-      			</geometry>
-    		</visual>
-			<collision>
-      			<origin xyz="0 0 0"/>
-				<geometry>
-					<box size="0.01 0.01 0.01"/>
-				</geometry>
-    		</collision>
-  	</link>
-	<joint name="join1" type="fixed">
-    		<origin xyz="3.983 0 0.15" rpy="0 0 0"/>
-    		<parent link="origin"/>
-    		<child link="wall_1"/>
-  	</joint>
-  	<link name="wall_1">
-    		<inertial>
-      			<origin xyz="0 0 0" />
-      			<mass value="10.0" />
-      			<inertia  ixx="1.0" ixy="0"  ixz="0"  iyy="1.0"  iyz="0"  izz="1.0" />
-    		</inertial>
-    		<visual>
-      			<origin xyz="0 0 0"/>
-      			<geometry>
-					<box size="0.04 0.8 0.3" /> <!--wall 80, width = 4 cm, lenght = 80 cm, height = 30 cm-->
-      			</geometry>
-    		</visual>
-			<collision>
-      			<origin xyz="0 0 0"/>
-				<geometry>
-					<box size="0.04 0.8 0.3"/>
-				</geometry>
-    		</collision>
-  	</link>
-	<joint name="join2" type="fixed">
-    		<origin xyz="0 0.842 0" rpy="0 0 0"/>
-    		<parent link="wall_1"/>
-    		<child link="wall_2"/>
-  	</joint>
-  	<link name="wall_2">
-    		<inertial>
-      			<origin xyz="0 0 0" />
-      			<mass value="10.0" />
-      			<inertia  ixx="1.0" ixy="0.0"  ixz="0.0"  iyy="1.0"  iyz="0.0"  izz="1.0" />
-    		</inertial>
-    		<visual>
-      			<origin xyz="0 0 0"/>
-      			<geometry>
-					<box size="0.04 0.8 0.3" /> <!--wall 80, width = 4 cm, lenght = 80 cm, height = 30 cm-->
-      			</geometry>
-    		</visual>
-			<collision>
-      			<origin xyz="0 0 0"/>
-				<geometry>
-					<box size="0.04 0.8 0.3"/>
-				</geometry>
-    		</collision>
-  	</link>
-  	<joint name="join3" type="fixed">
-    		<origin xyz="-0.580 0.421 0" rpy="0 0 1.570796"/>
-    		<parent link="wall_2"/>
-    		<child link="wall_3"/>
-  	</joint>
-  	<link name="wall_3">
-    		<inertial>
-      			<origin xyz="0 0 0" />
-      			<mass value="10.0" />
-      			<inertia  ixx="1.0" ixy="0.0"  ixz="0.0"  iyy="1.0"  iyz="0.0"  izz="1.0" />
-    		</inertial>
-    		<visual>
-      			<origin xyz="0 0 0"/>
-      			<geometry>
-					<box size="0.04 1.2 0.3" /> <!--wall 120, width = 4 cm, lenght = 120 cm, height = 30 cm-->
-      			</geometry>
-    		</visual>
-			<collision>
-      			<origin xyz="0 0 0"/>
-				<geometry>
-					<box size="0.04 1.2 0.3"/>
-				</geometry>
-    		</collision>
-  	</link>
-  	<joint name="join4" type="fixed">
-    		<origin xyz="0 1.201 0" rpy="0 0 0"/>
-    		<parent link="wall_3"/>
-    		<child link="wall_4"/>
-  	</joint>
-  	<link name="wall_4">
-    		<inertial>
-      			<origin xyz="0 0 0" />
-      			<mass value="0" />
-				<inertia  ixx="0" ixy="0"  ixz="0"  iyy="0"  iyz="0"  izz="0" />
-      			<!--inertia  ixx="1.0" ixy="0.0"  ixz="0.0"  iyy="1.0"  iyz="0.0"  izz="1.0" /-->
-    		</inertial>
-    		<visual>
-      			<origin xyz="0 0 0"/>
-      			<geometry>
-					<box size="0.01 0.01 0.01" /> <!--Insert 120 wall here for closed arena-->
-					<!--box size="0.04 1.2 0.3" /--> <!--wall 120, width = 4 cm, lenght = 120 cm, height = 30 cm-->
-      			</geometry>
-    		</visual>
-            <!-- Uncomment following block for closed arena -->
-			<!-- <collision> -->
-            <!-- <origin xyz="0 0 0"/> -->
-			<!-- 	<geometry> -->
-			<!-- 		<box size="0.04 0.8 0.3"/> -->
-			<!-- 	</geometry> -->
-    		<!-- </collision> -->
-  	</link>
-  	<joint name="join5" type="fixed">
-    		<origin xyz="0 1.201 0" rpy="0 0 0"/>
-    		<parent link="wall_4"/>
-    		<child link="wall_5"/>
-  	</joint>
-  	<link name="wall_5">
-    		<inertial>
-      			<origin xyz="0 0 0" />
-      			<mass value="0" />
-				<inertia  ixx="0" ixy="0"  ixz="0"  iyy="0"  iyz="0"  izz="0" />
-      			<!--inertia  ixx="1.0" ixy="0.0"  ixz="0.0"  iyy="1.0"  iyz="0.0"  izz="1.0" /-->
-    		</inertial>
-    		<visual>
-      			<origin xyz="0 0 0"/>
-      			<geometry>
-					<box size="0.01 0.01 0.01" /> <!--Insert 80 wall here for closed arena-->
-					<!--box size="0.04 0.8 0.3" /--> <!--wall 80, width = 4 cm, lenght = 80 cm, height = 30 cm-->
-      			</geometry>
-    		</visual>
-            <!-- Uncomment following block for closed arena -->
-			<!-- <collision> -->
-            <!-- <origin xyz="0 0 0"/> -->
-			<!-- 	<geometry> -->
-			<!-- 		<box size="0.04 0.8 0.3"/> -->
-			<!-- 	</geometry> -->
-    		<!-- </collision> -->
-  	</link>
-  	<joint name="join6" type="fixed">
-    		<origin xyz="0 0.801 0" rpy="0 0 0"/>
-    		<parent link="wall_5"/>
-    		<child link="wall_6"/>
-  	</joint>
-  	<link name="wall_6">
-    		<inertial>
-      			<origin xyz="0 0 0" />
-      			<mass value="10.0" />
-      			<inertia  ixx="1.0" ixy="0.0"  ixz="0.0"  iyy="1.0"  iyz="0.0"  izz="1.0" />
-    		</inertial>
-    		<visual>
-      			<origin xyz="0 0 0"/>
-      			<geometry>
-					<box size="0.04 0.8 0.3" /> <!--wall 80, width = 4 cm, lenght = 80 cm, height = 30 cm-->
-      			</geometry>
-    		</visual>
-			<collision>
-      			<origin xyz="0 0 0"/>
-				<geometry>
-					<box size="0.04 0.8 0.3"/>
-				</geometry>
-    		</collision>
-  	</link>
-  	<joint name="join7" type="fixed">
-			<origin xyz="-0.421 0.380 0" rpy="0 0 -1.570796"/>
-    		<parent link="wall_6"/>
-    		<child link="wall_7"/>
-  	</joint>
-  	<link name="wall_7">
-    		<inertial>
-      			<origin xyz="0 0 0" />
-      			<mass value="10.0" />
-      			<inertia  ixx="1.0" ixy="0.0"  ixz="0.0"  iyy="1.0"  iyz="0.0"  izz="1.0" />
-    		</inertial>
-    		<visual>
-      			<origin xyz="0 0 0"/>
-      			<geometry>
-					<box size="0.04 0.8 0.3" /> <!--wall 80, width = 4 cm, lenght = 80 cm, height = 30 cm-->
-      			</geometry>
-    		</visual>
-			<collision>
-      			<origin xyz="0 0 0"/>
-				<geometry>
-					<box size="0.04 0.8 0.3"/>
-				</geometry>
-    		</collision>
-  	</link>
-  	<joint name="join8" type="fixed">
-			<origin xyz="-0.421 0.129 -0.1" rpy="0 0 -1.570796"/>
-    		<parent link="wall_6"/>
-    		<child link="wall_8"/>
-  	</joint>
-  	<link name="wall_8">
-    		<inertial>
-      			<origin xyz="0 0 0" />
-      			<mass value="10.0" />
-      			<inertia  ixx="1.0" ixy="0.0"  ixz="0.0"  iyy="1.0"  iyz="0.0"  izz="1.0" />
-    		</inertial>
-    		<visual>
-      			<origin xyz="0 0 0"/>
-      			<geometry>
-					<box size="0.46 0.8 0.1" /> <!--platform, width = 46 cm, lenght = 80 cm, height = 10 cm-->
-      			</geometry>
-    		</visual>
-			<collision>
-      			<origin xyz="0 0 0"/>
-				<geometry>
-					<box size="0.46 0.8 0.1"/>
-				</geometry>
-    		</collision>
-  	</link>
-  	<joint name="join9" type="fixed">
-			<origin xyz="0 -0.842 0" rpy="0 0 0"/>
-    		<parent link="wall_1"/>
-    		<child link="wall_9"/>
-  	</joint>
-  	<link name="wall_9">
-    		<inertial>
-      			<origin xyz="0 0 0" />
-      			<mass value="10.0" />
-      			<inertia  ixx="1.0" ixy="0.0"  ixz="0.0"  iyy="1.0"  iyz="0.0"  izz="1.0" />
-    		</inertial>
-    		<visual>
-      			<origin xyz="0 0 0"/>
-      			<geometry>
-					<box size="0.04 0.8 0.3" /> <!--wall 80, width = 4 cm, lenght = 80 cm, height = 30 cm-->
-      			</geometry>
-    		</visual>
-			<collision>
-      			<origin xyz="0 0 0"/>
-				<geometry>
-					<box size="0.04 0.8 0.3"/>
-				</geometry>
-    		</collision>
-  	</link>
-  	<joint name="join10" type="fixed">
-			<origin xyz="-0.580 -0.421 0" rpy="0 0 1.570796"/>
-    		<parent link="wall_9"/>
-    		<child link="wall_10"/>
-  	</joint>
-  	<link name="wall_10">
-    		<inertial>
-      			<origin xyz="0 0 0" />
-      			<mass value="10.0" />
-      			<inertia  ixx="1.0" ixy="0.0"  ixz="0.0"  iyy="1.0"  iyz="0.0"  izz="1.0" />
-    		</inertial>
-    		<visual>
-      			<origin xyz="0 0 0"/>
-      			<geometry>
-					<box size="0.04 1.2 0.3" /> <!--wall 120, width = 4 cm, lenght = 120 cm, height = 30 cm-->
-      			</geometry>
-    		</visual>
-			<collision>
-      			<origin xyz="0 0 0"/>
-				<geometry>
-					<box size="0.04 1.2 0.3"/>
-				</geometry>
-    		</collision>
-  	</link>
-  	<joint name="join11" type="fixed">
-			<origin xyz="0 1.201 0" rpy="0 0 0"/>
-    		<parent link="wall_10"/>
-    		<child link="wall_11"/>
-  	</joint>
-  	<link name="wall_11">
-    		<inertial>
-      			<origin xyz="0 0 0" />
-      			<mass value="0" />
-				<inertia  ixx="0" ixy="0"  ixz="0"  iyy="0"  iyz="0"  izz="0" />
-      			<!--inertia  ixx="1.0" ixy="0.0"  ixz="0.0"  iyy="1.0"  iyz="0.0"  izz="1.0" /-->
-    		</inertial>
-    		<visual>
-      			<origin xyz="0 0 0"/>
-      			<geometry>
-					<box size="0.01 0.01 0.01" /> <!--Insert 120 wall here for closed arena-->
-					<!--box size="0.04 1.2 0.3" /--> <!--wall 120, width = 4 cm, lenght = 120 cm, height = 30 cm-->
-      			</geometry>
-    		</visual>
-            <!-- Uncomment following block for closed arena -->
-			<!-- <collision> -->
-            <!-- <origin xyz="0 0 0"/> -->
-			<!-- 	<geometry> -->
-			<!-- 		<box size="0.04 0.8 0.3"/> -->
-			<!-- 	</geometry> -->
-    		<!-- </collision> -->
-  	</link>
-  	<joint name="join12" type="fixed">
-			<origin xyz="0 1.201 0" rpy="0 0 0"/>
-    		<parent link="wall_11"/>
-    		<child link="wall_12"/>
-  	</joint>
-  	<link name="wall_12">
-    		<inertial>
-      			<origin xyz="0 0 0" />
-      			<mass value="0" />
-				<inertia  ixx="0" ixy="0"  ixz="0"  iyy="0"  iyz="0"  izz="0" />
-      			<!--inertia  ixx="1.0" ixy="0.0"  ixz="0.0"  iyy="1.0"  iyz="0.0"  izz="1.0" /-->
-    		</inertial>
-    		<visual>
-      			<origin xyz="0 0 0"/>
-      			<geometry>
-					<box size="0.01 0.01 0.01" /> <!--Insert 80 wall here for closed arena-->
-					<!--box size="0.04 0.8 0.3" /--> <!--wall 80, width = 4 cm, lenght = 80 cm, height = 30 cm-->
-      			</geometry>
-    		</visual>
-            <!-- Uncomment following block for closed arena -->
-			<!-- <collision> -->
-            <!-- <origin xyz="0 0 0"/> -->
-			<!-- 	<geometry> -->
-			<!-- 		<box size="0.04 0.8 0.3"/> -->
-			<!-- 	</geometry> -->
-    		<!-- </collision> -->
-  	</link>
-  	<joint name="join13" type="fixed">
-			<origin xyz="0 0.801 0" rpy="0 0 0"/>
-    		<parent link="wall_12"/>
-    		<child link="wall_13"/>
-  	</joint>
-  	<link name="wall_13">
-    		<inertial>
-      			<origin xyz="0 0 0" />
-      			<mass value="10.0" />
-      			<inertia  ixx="1.0" ixy="0.0"  ixz="0.0"  iyy="1.0"  iyz="0.0"  izz="1.0" />
-    		</inertial>
-    		<visual>
-      			<origin xyz="0 0 0"/>
-      			<geometry>
-					<box size="0.04 0.8 0.3" /> <!--wall 80, width = 4 cm, lenght = 80 cm, height = 30 cm-->
-      			</geometry>
-    		</visual>
-			<collision>
-      			<origin xyz="0 0 0"/>
-				<geometry>
-					<box size="0.04 0.8 0.3"/>
-				</geometry>
-    		</collision>
-  	</link>
-  	<joint name="join14" type="fixed">
-			<origin xyz="0.421 0.380 0" rpy="0 0 -1.570796"/>
-    		<parent link="wall_13"/>
-    		<child link="wall_14"/>
-  	</joint>
-  	<link name="wall_14">
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