Commit message: [description] update masses

File: mcr_common/mcr_description/urdf/fingers/festo_finger_dhas-gf-shm.urdf.xacro (robot description, xacro)
@@ -13,5 +13,5 @@
       <inertial>
         <origin xyz="0 0 0" rpy="0 0 0"/>
-        <mass value="0.1"/>
+        <mass value="0.015"/>
         <inertia ixx="0.01" ixy="0" ixz="0" iyy="0.01" iyz="0" izz="0.01" />
       </inertial>

File: mcr_common/mcr_description/urdf/sensors/intel_realsense_f200_camera.urdf.xacro (robot description, xacro)
@@ -10,5 +10,5 @@
 	<link name="${parent}_${suffix}_frame">
 	  <inertial>
-		<mass value="0.01" />
+		<mass value="0.0001" />
 		<origin xyz="0 0 0" />
 		<inertia ixx="0.1" ixy="0" ixz="0" iyy="0.1" iyz="0" izz="0.1" />
@@ -24,5 +24,5 @@
     <link name="${name}_link">
       <inertial>
-        <mass value="0.1" />
+        <mass value="0.170" />
         <origin xyz="0 0 0" rpy="0 0 0"/>
         <inertia ixx="0.0001" ixy="0" ixz="0" iyy="0.0001" iyz="0" izz="0.0001" />

Commit message: fix property and insert_block tags in URDF files

File: mcr_common/mcr_description/urdf/fingers/festo_finger_dhas-gf-shm.urdf.xacro (robot description, xacro)
@@ -6,5 +6,5 @@
   <xacro:macro name="festo_finger_DHAS-GF-shm" params="parent name *origin">
     <joint name="${name}_joint" type="fixed" >
-      <insert_block name="origin" />
+      <xacro:insert_block name="origin" />
       <parent link="${parent}" />
       <child link="${name}_link" />

File: mcr_common/mcr_description/urdf/motors/dynamixel_bracket_fp04-f2.urdf.xacro (robot description, xacro)
@@ -6,5 +6,5 @@
   <xacro:macro name="dynamixel_bracket_FP04-F2" params="parent name *origin">
     <joint name="${name}_joint" type="fixed" >
-      <insert_block name="origin" />
+      <xacro:insert_block name="origin" />
       <parent link="${parent}" />
       <child link="${name}_link" />

File: mcr_common/mcr_description/urdf/motors/dynamixel_motor_ax-12a.urdf.xacro (robot description, xacro)
@@ -8,5 +8,5 @@
   <xacro:macro name="dynamixel_motor_AX-12A" params="parent name *origin motor_direction position_offset">
     <joint name="${name}_base_joint" type="fixed" >
-      <insert_block name="origin" />
+      <xacro:insert_block name="origin" />
       <parent link="${parent}" />
       <child link="${name}_base_link" />

File: mcr_common/mcr_description/urdf/sensors/intel_realsense_f200_camera.urdf.xacro (robot description, xacro)
@@ -5,7 +5,7 @@
        xmlns:xacro="http://ros.org/wiki/xacro">
   <xacro:include filename="$(find mcr_description)/urdf/sensors/intel_realsense_f200_camera.gazebo.xacro" />
-  <property name="eye_x_offset" value="-0.015" />
-  <property name="eye_y_offset" value="0.024" />
-  <property name="eye_z_offset" value="0.018" />
+  <xacro:property name="eye_x_offset" value="-0.015" />
+  <xacro:property name="eye_y_offset" value="0.024" />
+  <xacro:property name="eye_z_offset" value="0.018" />
   <xacro:macro name="intel_realsense_f200_eye" params="suffix parent *origin">
 	<link name="${parent}_${suffix}_frame">
